File: MFRC522 Board/Alt/PCB Nodev3 v1.3.kicad_pcb (KiCad board)
At the start: 2 copper layers, 120 x 50 mm, 56 parts, among them P1 ESP32 NODEMCU DEVKIT1 LEFT HE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, P2 ESP32 NODEMCU DEVKIT1 RIGHT H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, Q1 Q_NPN_BEC, Q2 Q_NPN_BEC, U1 MFRC522, U2 3,0, U3 3,0, U4 3,0, U5 3,0, U6 Tooling Hole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

Commit message: moved stuff to allow multiple boards in the same repo
Parts:
- removed 1: OSHW-LOGOM, easyeda:OSHWLOGO_TOP_0.2
- removed C13: 22nF, Capacitor_SMD:C_0603_1608Metric
- removed C14: 10nF, Capacitor_SMD:C_0603_1608Metric
- removed Q1: Q_NPN_BEC, Package_TO_SOT_SMD:SOT-23
- removed R12: 68K, Resistor_SMD:R_0603_1608Metric
- removed R13: 2K, Resistor_SMD:R_0603_1608Metric
- removed R15: 9.1K, Resistor_SMD:R_0603_1608Metric
- removed R17: 3.3K, Resistor_SMD:R_0603_1608Metric
- removed R7, R8: 18K, Resistor_SMD:R_0603_1608Metric
- removed R9: 68, Resistor_SMD:R_0603_1608Metric
- removed U2, U3, U4, U5: 3,0, easyeda:MOUNTINGHOLE_3.0
- removed U6, U7, U8: Tooling Hole, easyeda:TOOLING_HOLE_JLCPCB
- removed U9: NE555, Package_SO:SOIC-8_3.9x4.9mm_P1.27mm
- R16: value 200 -> 240
- moved R16 37.1 mm to (130.9, 100.3), turned to 180 degrees
Connections:
- P1 pad 1: Net-(P1-Pad1) -> (no net)
- P1 pad 12: Net-(P1-Pad12) -> (no net)
- P1 pad 13: Net-(P1-Pad13) -> (no net)
- P1 pad 2: Net-(P1-Pad2) -> (no net)
- P1 pad 3: Net-(P1-Pad3) -> (no net)
- P1 pad 4: /GPIO-TH -> (no net)
- P1 pad 7: Net-(P1-Pad7) -> (no net)
- P2 pad 1: Net-(P2-Pad1) -> (no net)
- P2 pad 11: Net-(P2-Pad11) -> (no net)
- P2 pad 12: Net-(P2-Pad12) -> (no net)
- P2 pad 13: Net-(P2-Pad13) -> (no net)
- P2 pad 15: Net-(P2-Pad15) -> (no net)
- P2 pad 2: Net-(P2-Pad2) -> (no net)
- P2 pad 4: Net-(P2-Pad4) -> (no net)
- P2 pad 5: Net-(P2-Pad5) -> (no net)
- P2 pad 8: Net-(P2-Pad8) -> /GPIO-TH
- R16 pad 1: /BZROSC -> /GPIO-TH
- U1 pad 1: Net-(U1-Pad1) -> (no net)
- U1 pad 19: Net-(U1-Pad19) -> (no net)
- U1 pad 20: Net-(U1-Pad20) -> (no net)
- U1 pad 25: Net-(U1-Pad25) -> (no net)
- U1 pad 26: Net-(U1-Pad26) -> (no net)
- U1 pad 27: Net-(U1-Pad27) -> (no net)
- U1 pad 28: Net-(U1-Pad28) -> (no net)
- U1 pad 7: Net-(U1-Pad7) -> (no net)
- U1 pad 8: Net-(U1-Pad8) -> (no net)
- U1 pad 9: Net-(U1-Pad9) -> (no net)
Routing:
- net Net-(Q2-Pad1): track 100.3 -> 6.19 mm, vias 2 -> 0
- net +5V: track 106.9 -> 50.6 mm, vias 4 -> 2
- net Net-(C13-Pad2): track 41.8 -> 0.00 mm, vias 2 -> 0
- net Net-(Q1-Pad2): track 41.1 -> 0.00 mm, vias 4 -> 0
- net Net-(R12-Pad2): track 8.85 -> 0.00 mm
- net GND: track 859.9 -> 852.4 mm, vias 21 -> 19
- net /BZROSC: track 6.93 -> 0.00 mm
- net Net-(R7-Pad1): track 4.48 -> 0.00 mm
- net Net-(Q1-Pad1): track 2.23 -> 0.00 mm
- net Net-(R12-Pad1): track 1.96 -> 0.00 mm
Other:
- rule via_min_size: 0.4 -> 0.45
- board text added: "GND|+5V"
- board text added: "MicroUSB on this side"
