File: MFRC522 Board/v1.3/PCB Nodev3 v1.3.kicad_pcb (KiCad board)
At the start: 2 copper layers, 120 x 50 mm, 56 parts, among them P1 ESP32 NODEMCU DEVKIT1 LEFT HE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, P2 ESP32 NODEMCU DEVKIT1 RIGHT H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, Q1 Q_NPN_BEC, Q2 Q_NPN_BEC, U1 MFRC522, U2 3,0, U3 3,0, U4 3,0, U5 3,0, U6 Tooling Hole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

Commit message: mod.
Routing:
- net Net-(Q2-Pad1): track 100.3 -> 101.0 mm
Changed lines of the file:
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@@
   (segment (start 130.409 65.298) (end 130.086 65.621) (width 0.381) (layer F.Cu) (net 43))
   (segment (start 130.086 65.621) (end 130.086 66.675) (width 0.381) (layer F.Cu) (net 43))
-  (segment (start 113.411 68.834) (end 153.289 68.834) (width 0.508) (layer B.Cu) (net 44))
-  (segment (start 153.289 68.834) (end 154.051 69.596) (width 0.508) (layer B.Cu) (net 44))
-  (segment (start 154.051 69.596) (end 154.051 95.377) (width 0.508) (layer B.Cu) (net 44))
-  (segment (start 154.051 95.377) (end 152.908 96.52) (width 0.508) (layer B.Cu) (net 44))
-  (segment (start 152.908 96.52) (end 141.097 96.52) (width 0.508) (layer B.Cu) (net 44))
-  (segment (start 141.097 96.52) (end 138.43 99.187) (width 0.508) (layer B.Cu) (net 44))
-  (segment (start 138.43 99.187) (end 129.794 99.187) (width 0.508) (layer B.Cu) (net 44))
   (segment (start 112.052 68.834) (end 113.411 68.834) (width 0.508) (layer F.Cu) (net 44))
   (via (at 129.794 99.187) (size 0.61) (drill 0.305) (layers F.Cu B.Cu) (net 44))
@@
   (segment (start 129.794 99.187) (end 128.59 100.391) (width 0.508) (layer F.Cu) (net 44))
   (segment (start 128.59 100.391) (end 123.936 100.391) (width 0.508) (layer F.Cu) (net 44))
+  (segment (start 138.43 99.187) (end 129.794 99.187) (width 0.508) (layer B.Cu) (net 44))
+  (segment (start 140.716 96.901) (end 138.43 99.187) (width 0.508) (layer B.Cu) (net 44))
+  (segment (start 153.6192 68.834) (end 154.1272 69.342) (width 0.508) (layer B.Cu) (net 44))
+  (segment (start 113.411 68.834) (end 153.6192 68.834) (width 0.508) (layer B.Cu) (net 44))
+  (segment (start 154.1272 69.342) (end 154.1272 96.0755) (width 0.508) (layer B.Cu) (net 44))
+  (segment (start 154.1272 96.0755) (end 153.3017 96.901) (width 0.508) (layer B.Cu) (net 44))
+  (segment (start 153.3017 96.901) (end 140.716 96.901) (width 0.508) (layer B.Cu) (net 44))
   (segment (start 121.196 62.865) (end 123.152 62.865) (width 0.381) (layer F.Cu) (net 45))
   (segment (start 123.152 62.865) (end 123.317 63.03) (width 0.381) (layer F.Cu) (net 45))
