File: In Development/MFRC522 Board/v1.31/PCB Nodev3 v1.31.sch (KiCad schematic (older format))
At the start: 37 parts, among them P1 ESP32 NODEMCU DEVKIT1 LEFT HE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, P2 ESP32 NODEMCU DEVKIT1 RIGHT H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, Q2 Q_NPN_BEC, U1 MFRC522, Y1 27.12 MHz

Commit message: redrew, and anotatted some caps and leds
Parts:
- added H1, H2, H3, H4: MountingHole, MountingHole:MountingHole_3.2mm_M3, symbol Mechanical:MountingHole
- added H5, H6, H7: ToolingHole, Custom:TOOLING_HOLE_JLCPCB_SMT, symbol Mechanical:ToolingHole
- added LG1: Logo_Open_Hardware_Small, Custom:OSHWLOGO_TOP_0.2, symbol Graphic:Logo_Open_Hardware_Small
- C3, C4: value C_Small -> 1uF
- LED1: value LED -> LED_GREEN
- LED2: value LED -> LED_BLUE
Changed lines of the file:
@@
 	0    1    1    0
-$EndComp
-$Comp
-L RF_Module:MFRC522 U1
-U 1 1 5EA9A706
-P 4750 3250
-F 0 "U1" H 4550 3350 50  0000 L CNN
-F 1 "MFRC522" H 4550 3250 50  0000 L CNN
-F 2 "Package_DFN_QFN:QFN-32-1EP_5x5mm_P0.5mm_EP3.1x3.1mm" H 4750 3250 50  0001 C CNN
-F 3 "https://www.nxp.com/docs/en/data-sheet/MFRC522.pdf" H 4750 3250 50  0001 C CNN
-	1    4750 3250
-	1    0    0    -1
 $EndComp
 Wire Wire Line
@@
 P 2600 6300
 F 0 "LED2" V 2639 6183 50  0000 R CNN
-F 1 "LED" V 2548 6183 50  0000 R CNN
+F 1 "LED_BLUE" V 2548 6183 50  0000 R CNN
 F 2 "LED_SMD:LED_0603_1608Metric" H 2600 6300 50  0001 C CNN
 F 3 "~" H 2600 6300 50  0001 C CNN
@@
 P 1500 6300
 F 0 "LED1" V 1539 6183 50  0000 R CNN
-F 1 "LED" V 1448 6183 50  0000 R CNN
+F 1 "LED_GREEN" V 1448 6183 50  0000 R CNN
 F 2 "LED_SMD:LED_0603_1608Metric" H 1500 6300 50  0001 C CNN
 F 3 "~" H 1500 6300 50  0001 C CNN
@@
 P 1750 4800
 F 0 "C3" H 1842 4846 50  0000 L CNN
-F 1 "C_Small" H 1842 4755 50  0000 L CNN
+F 1 "1uF" H 1842 4755 50  0000 L CNN
 F 2 "Capacitor_SMD:C_0805_2012Metric" H 1750 4800 50  0001 C CNN
 F 3 "~" H 1750 4800 50  0001 C CNN
@@
 P 2350 4800
 F 0 "C4" H 2442 4846 50  0000 L CNN
-F 1 "C_Small" H 2442 4755 50  0000 L CNN
+F 1 "1uF" H 2442 4755 50  0000 L CNN
 F 2 "Capacitor_SMD:C_0805_2012Metric" H 2350 4800 50  0001 C CNN
 F 3 "~" H 2350 4800 50  0001 C CNN
@@
 Text Notes 7050 7100 0    50   ~ 0
 Designed by Probably an Asian\nAntenna design and matching circuit adapted from Adafruit's PN532 Breakout Board\n\nhttps://github.com/innexgo/pcb\n\nINNEXGO LLC.
+$Comp
+L Mechanical:MountingHole H1
+U 1 1 5EAF8031
+P 8100 800
+F 0 "H1" H 8328 846 50  0000 L CNN
+F 1 "MountingHole" H 8328 755 50  0000 L CNN
+F 2 "MountingHole:MountingHole_3.2mm_M3" H 8100 800 50  0001 C CNN
+F 3 "~" H 8100 800 50  0001 C CNN
+	1    8100 800
+	1    0    0    -1
+$EndComp
+$Comp
+L Mechanical:MountingHole H3
+U 1 1 5EAF898E
+P 8100 1100
+F 0 "H3" H 8328 1146 50  0000 L CNN
+F 1 "MountingHole" H 8328 1055 50  0000 L CNN
+F 2 "MountingHole:MountingHole_3.2mm_M3" H 8100 1100 50  0001 C CNN
+F 3 "~" H 8100 1100 50  0001 C CNN
+	1    8100 1100
+	1    0    0    -1
+$EndComp
+$Comp
+L Mechanical:MountingHole H2
+U 1 1 5EAF83C7
+P 8950 800
+F 0 "H2" H 9178 846 50  0000 L CNN
+F 1 "MountingHole" H 9178 755 50  0000 L CNN
+F 2 "MountingHole:MountingHole_3.2mm_M3" H 8950 800 50  0001 C CNN
+F 3 "~" H 8950 800 50  0001 C CNN
+	1    8950 800
+	1    0    0    -1
+$EndComp
+$Comp
+L Mechanical:MountingHole H4
+U 1 1 5EAF9734
+P 8950 1100
+F 0 "H4" H 9178 1146 50  0000 L CNN
+F 1 "MountingHole" H 9178 1055 50  0000 L CNN
+F 2 "MountingHole:MountingHole_3.2mm_M3" H 8950 1100 50  0001 C CNN
+F 3 "~" H 8950 1100 50  0001 C CNN
+	1    8950 1100
+	1    0    0    -1
+$EndComp
+$Comp
+L Mechanical:ToolingHole H5
+U 1 1 5EB15676
+P 8100 1400
+F 0 "H5" H 8185 1446 50  0000 L CNN
+F 1 "ToolingHole" H 8185 1355 50  0000 L CNN
+F 2 "Custom:TOOLING_HOLE_JLCPCB_SMT" H 8100 1400 50  0001 C CNN
+F 3 "~" H 8100 1400 50  0001 C CNN
+	1    8100 1400
+	1    0    0    -1
+$EndComp
+$Comp
+L Mechanical:ToolingHole H7
+U 1 1 5EAF7D4C
+P 8850 1400
+F 0 "H7" H 8935 1446 50  0000 L CNN
+F 1 "ToolingHole" H 8935 1355 50  0000 L CNN
+F 2 "Custom:TOOLING_HOLE_JLCPCB_SMT" H 8850 1400 50  0001 C CNN
+F 3 "~" H 8850 1400 50  0001 C CNN
+	1    8850 1400
+	1    0    0    -1
+$EndComp
+$Comp
+L Mechanical:ToolingHole H6
+U 1 1 5EAF80D3
+P 8100 1650
+F 0 "H6" H 8185 1696 50  0000 L CNN
+F 1 "ToolingHole" H 8185 1605 50  0000 L CNN
+F 2 "Custom:TOOLING_HOLE_JLCPCB_SMT" H 8100 1650 50  0001 C CNN
+F 3 "~" H 8100 1650 50  0001 C CNN
+	1    8100 1650
+	1    0    0    -1
+$EndComp
+$Comp
+L Graphic:Logo_Open_Hardware_Small LG1
+U 1 1 5EB0E76A
+P 8950 1750
+F 0 "LG1" H 8950 2025 50  0001 C CNN
+F 1 "Logo_Open_Hardware_Small" H 8950 1525 50  0001 C CNN
+F 2 "Custom:OSHWLOGO_TOP_0.2" H 8950 1750 50  0001 C CNN
+F 3 "~" H 8950 1750 50  0001 C CNN
+	1    8950 1750
+	1    0    0    -1
+$EndComp
+$Comp
+L RF_Module:MFRC522 U1
+U 1 1 5EA9A706
+P 4750 3250
+F 0 "U1" H 4550 3350 50  0000 L CNN
+F 1 "MFRC522" H 4550 3250 50  0000 L CNN
+F 2 "Package_DFN_QFN:QFN-32-1EP_5x5mm_P0.5mm_EP3.1x3.1mm" H 4750 3250 50  0001 C CNN
+F 3 "https://www.nxp.com/docs/en/data-sheet/MFRC522.pdf" H 4750 3250 50  0001 C CNN
+	1    4750 3250
+	1    0    0    -1
+$EndComp
 $EndSCHEMATC
