File: In Development/MFRC522 Board/Latest/MFRC522 PCB Nodev3.sch (KiCad schematic (older format))
At the start: 45 parts, among them P1 ESP32 NODEMCU DEVKIT1 LEFT HE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, P2 ESP32 NODEMCU DEVKIT1 RIGHT H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, Q2 Q_NPN_BEC, U1 MFRC522, Y1 27.12 MHz

Commit message: prep for ordering
Parts:
- U1: symbol RF_Module:MFRC522 -> Custom:MFRC522
Changed lines of the file:
@@
 $EndComp
 $Comp
-L RF_Module:MFRC522 U1
+L Custom:MFRC522 U1
 U 1 1 5EA9A706
 P 4750 3250
