File: In Development/MFRC522 Board/Latest/MFRC522 PCB Nodev2.kicad_pcb (KiCad board)
At the start: 2 copper layers, 120 x 50 mm, 45 parts, among them P1 ESP32 NODEMCU DEVKIT1 LEFT HE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, P2 ESP32 NODEMCU DEVKIT1 RIGHT H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, Q2 Q_NPN_BEC, U1 MFRC522, Y1 27.12 MHz

Commit message: In production.
Parts:
- added R20: R_Axial, Resistor_THT:R_Axial_DIN0309_L9.0mm_D3.2mm_P12.70mm_Horizontal, F.Cu at (136.7, 98.0)
- C10, C16: footprint Capacitor_SMD:C_0805_2012Metric -> Capacitor_SMD:C_0603_1608Metric
- C3, C4: value C_Small -> 1uF
- LED1: value LED -> LED_GREEN
- LED2: value LED -> LED_BLUE
- moved L2 1.62 mm to (116.8, 90.1)
- moved C8 0.49 mm to (112.3, 78.3)
- moved C10 0.44 mm to (110.0, 78.3)
- moved L1 0.40 mm to (115.0, 78.3)
- moved C16 0.38 mm to (110.0, 85.8)
- moved C11 0.34 mm to (107.5, 84.3)
- moved R5 0.34 mm to (105.0, 78.3)
- moved R6 0.34 mm to (105.0, 85.8)
- moved C5 0.33 mm to (107.5, 79.8)
- moved C7 0.25 mm to (112.3, 85.8)
- moved C12 0.25 mm to (120.8, 83.8)
- moved R11 0.25 mm to (118.3, 85.8)
- moved R10 0.24 mm to (114.3, 85.8)
- moved C15 0.24 mm to (116.3, 85.8)
- moved TP1 0.17 mm to (105.0, 75.8)
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Routing:
- net Net-(BZ1-Pad1): track 21.2 -> 31.6 mm, vias 0 -> 1
- net Net-(L2-Pad1): track 19.9 -> 18.2 mm
- net GND: track 852.9 -> 852.4 mm, vias 23 -> 20
- removed copper zone on F.Cu, net +3V3
Other:
- board text added: "JLCJLCJLCJLC"
