File: In Development/MFRC522 Board/Latest/MFRC522 PCB Nodev2.sch (KiCad schematic (older format))
At the start: 46 parts, among them P1 ESP32 NODEMCU DEVKIT1 LEFT HE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, P2 ESP32 NODEMCU DEVKIT1 RIGHT H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, Q2 Q_NPN_BEC, U1 MFRC522, Y1 27.12 MHz

Commit message: update for ESP32, so not actually Node anymore
Parts:
- H5, H6, H7: symbol Mechanical:ToolingHole -> MFRC522-PCB-Nodev2-rescue:ToolingHole-Mechanical
- U1: symbol Custom:MFRC522 -> MFRC522-PCB-Nodev2-rescue:MFRC522-Custom
Connections:
- net +3V3: now also P1.10 (Pin_10); no longer P1.11 (Pin_11)
- net IRQ: now also P1.9 (Pin_9); no longer P1.5 (Pin_5)
- net MISO: now also P1.6 (Pin_6); no longer P1.8 (Pin_8)
- net MOSI: now also P1.7 (Pin_7); no longer P1.6 (Pin_6)
- net SCK: now also P1.8 (Pin_8); no longer P1.9 (Pin_9)
- net at C15.1, R11.1, U1.17 (RX): no longer U1.33 (UNC)
Changed lines of the file:
@@
 	1000 1300 1650 1300
-Wire Wire Line
-	1000 1400 1650 1400
 Wire Wire Line
 	1000 1500 1650 1500
@@
 NoConn ~ 1650 1100
 NoConn ~ 1650 1200
-Text HLabel 1650 1500 2    50   Output ~ 0
+Text HLabel 1650 1600 2    50   Output ~ 0
 SCK
-Text HLabel 1650 1600 2    50   Input ~ 0
+Text HLabel 1650 1800 2    50   Input ~ 0
 MISO
-Text HLabel 1650 1800 2    50   Output ~ 0
+Text HLabel 1650 1700 2    50   Output ~ 0
 MOSI
-NoConn ~ 1650 1700
 NoConn ~ 1650 2100
 NoConn ~ 1650 2200
 NoConn ~ 1650 2300
-Text HLabel 1650 1900 2    50   Output ~ 0
+Text HLabel 1650 1500 2    50   Output ~ 0
 IRQ
 Text HLabel 1650 3500 2    50   Output ~ 0
@@
 $EndComp
 $Comp
-L Mechanical:ToolingHole H5
+L MFRC522-PCB-Nodev2-rescue:ToolingHole-Mechanical H5
 U 1 1 5EB15676
 P 8100 1400
@@
 $EndComp
 $Comp
-L Mechanical:ToolingHole H7
+L MFRC522-PCB-Nodev2-rescue:ToolingHole-Mechanical H7
 U 1 1 5EAF7D4C
 P 8850 1400
@@
 $EndComp
 $Comp
-L Mechanical:ToolingHole H6
+L MFRC522-PCB-Nodev2-rescue:ToolingHole-Mechanical H6
 U 1 1 5EAF80D3
 P 8100 1650
@@
 $EndComp
 $Comp
-L Custom:MFRC522 U1
+L MFRC522-PCB-Nodev2-rescue:MFRC522-Custom U1
 U 1 1 5EA9A706
 P 4750 3250
@@
 NoConn ~ 1650 3900
 $Comp
-L power:+3.3V #PWR0106
-U 1 1 5F0CE5E6
-P 1650 1300
-F 0 "#PWR0106" H 1650 1150 50  0001 C CNN
-F 1 "+3.3V" V 1650 1400 50  0000 L CNN
-F 2 "" H 1650 1300 50  0001 C CNN
-F 3 "" H 1650 1300 50  0001 C CNN
-	1    1650 1300
-	0    1    1    0
-$EndComp
-NoConn ~ 1650 1400
-$Comp
-L power:+3.3V #PWR?
+L power:+3.3V #PWR0105
 U 1 1 5F09AE72
 P 5650 2450
-F 0 "#PWR?" H 5650 2300 50  0001 C CNN
+F 0 "#PWR0105" H 5650 2300 50  0001 C CNN
 F 1 "+3.3V" V 5665 2578 50  0000 L CNN
 F 2 "" H 5650 2450 50  0001 C CNN
@@
 $EndComp
 $Comp
-L power:+3.3V #PWR?
+L power:+3.3V #PWR0106
 U 1 1 5F09B301
 P 3700 3800
-F 0 "#PWR?" H 3700 3650 50  0001 C CNN
+F 0 "#PWR0106" H 3700 3650 50  0001 C CNN
 F 1 "+3.3V" H 3715 3928 50  0000 L CNN
 F 2 "" H 3700 3800 50  0001 C CNN
@@
 	-1   0    0    1
 $EndComp
+NoConn ~ 1650 1300
+$Comp
+L power:+3.3V #PWR0109
+U 1 1 60861254
+P 1650 1400
+F 0 "#PWR0109" H 1650 1250 50  0001 C CNN
+F 1 "+3.3V" V 1650 1500 50  0000 L CNN
+F 2 "" H 1650 1400 50  0001 C CNN
+F 3 "" H 1650 1400 50  0001 C CNN
+	1    1650 1400
+	0    1    1    0
+$EndComp
+Wire Wire Line
+	1000 1400 1650 1400
+NoConn ~ 1650 1900
 $EndSCHEMATC
