File: In Development/LED Timer/LED Timer/LED Timer.kicad_pcb (KiCad board)
At the start: 2 copper layers, 60 x 50 mm, 31 parts, among them J1 Barrel_Jack_Switch, J2 Conn_01x04_Male, J3 Conn_01x03_Female, SW1 DNP, U1 LM7805_TO252-2, U2 ESP-12E

Commit message: added a switch to dectect for soft-reset
Parts:
- added R13: 470, Resistor_SMD:R_0603_1608Metric, F.Cu at (143.0, 59.8)
- added R14: 12K, Resistor_SMD:R_0603_1608Metric, F.Cu at (143.8, 63.0)
- added SW2: SW2, Button_Switch_SMD:SW_SPST_EVQQ2, F.Cu at (149.2, 53.8)
- moved D5 1.50 mm to (157.2, 61.2)
- moved D6 1.50 mm to (157.2, 56.8)
- moved R9 1.50 mm to (157.2, 65.5)
- moved H1 1.41 mm to (111.0, 89.0)
- moved H2 1.41 mm to (149.0, 61.0)
- moved D2 0.50 mm to (140.8, 81.0)
Connections:
- J2 pad 2: /GPIO12 -> /GPIO13
- J2 pad 3: /GPIO12 -> /GPIO13
Routing:
- net /0VA: track 106.4 -> 148.6 mm
- net /GPIO12: track 36.6 -> 0.00 mm
- net /GPIO13: track 0.00 -> 35.7 mm
- net Net-(R13-Pad2): track 0.00 -> 16.3 mm
- net /GPIO5: track 0.00 -> 6.59 mm
- net +3.3VA: track 104.6 -> 108.6 mm
- net +12V: track 129.4 -> 128.2 mm
- net GND: track 51.5 -> 51.0 mm
Other:
- net class Default: clearance 0.2 -> 0.26
- rule trace_clearance: 0.2 -> 0.26
- board text added: "104"
- board text added: "1uF"
- board text added: "222"
- board text added: "224"

Commit message: mod.
Parts:
- removed D6: Red 2, LED_SMD:LED_0805_2012Metric
- R9: value 470 -> 510; footprint Resistor_SMD:R_0603_1608Metric -> Resistor_SMD:R_0805_2012Metric
- moved D4 3.02 mm to (130.0, 81.0)
- moved R8 2.57 mm to (126.5, 81.0)
- moved D5 2.00 mm to (157.2, 59.2)
- moved R9 1.56 mm to (157.2, 63.9)
Connections:
- D5 pad 1: Net-(D5-Pad1) -> GND
Routing:
- net Net-(D5-Pad1): track 2.62 -> 0.00 mm
- net /0VA: track 148.6 -> 150.8 mm, vias 5 -> 4
- net +3.3VA: track 108.6 -> 107.3 mm, vias 6 -> 5
- net +12V: track 128.2 -> 129.4 mm
- net Net-(D4-Pad2): track 2.28 -> 1.78 mm
- net GND: track 51.0 -> 51.5 mm

Commit message: added "Innexgo LLC" to the board.
Other:
- board text added: "Innexgo LLC"
Changed lines of the file:
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@@
   (general
     (thickness 1.6)
-    (drawings 459)
+    (drawings 460)
     (tracks 227)
     (zones 0)
@@
     )
   )
+  (gr_text "Innexgo LLC" (at 130 85) (layer B.SilkS)
+    (effects (font (size 3 3) (thickness 0.6)) (justify mirror))
+  )
   (gr_text 222 (at 110.25 56.25) (layer F.SilkS)

Commit message: In production.
Parts:
- removed the J2 at (105.0, 75.0)
- added FID1: Fiducial, Fiducial:Fiducial_0.5mm_Mask1mm, F.Cu at (110.0, 98.2)
- added FID2: Fiducial, Fiducial:Fiducial_0.5mm_Mask1mm, F.Cu at (140.0, 98.2)
- added FID3: Fiducial, Fiducial:Fiducial_0.5mm_Mask1mm, F.Cu at (135.0, 55.0)
- added J2: 4x_1.5mm_5.5mm_bare_copper, Custom:4x_1.5mm_5.5mm_bare_copper, B.Cu at (106.0, 75.0)
- added J2: Conn_01x04_Male, Custom:4x_1.5mm_5.5mm_bare_copper_+THT, F.Cu at (104.8, 75.0)
- added LOGO1: Logo_Open_Hardware_Small, Custom:OSHWLOGO_TOP_0.2_SC-ver, F.Cu at (145.0, 63.5)
- R1, R14, R2, R3, R4, R5: value 12K -> 10K
- R6: value 470 -> 22
- moved H2 55.6 mm to (105.0, 95.0), turned to 180 degrees
- moved H1 48.1 mm to (145.0, 55.0), turned to 180 degrees
- moved SW2 45.7 mm to (132.5, 96.2)
- moved R13 36.5 mm to (143.0, 96.2), turned to 180 degrees
- moved D5 27.7 mm to (141.8, 82.2), turned to 180 degrees
- moved C4 22.5 mm to (121.2, 79.5), turned to 0 degrees
- moved R9 21.5 mm to (146.0, 82.2), turned to 180 degrees
- moved D3 18.0 mm to (108.2, 82.2), turned to 0 degrees
- moved R6 17.0 mm to (104.5, 82.2), turned to 180 degrees
- moved C1 10.6 mm to (137.2, 82.2)
- moved R1 10.3 mm to (133.5, 66.8)
- moved R14 10.3 mm to (133.5, 62.8)
- moved R2 10.3 mm to (133.5, 68.8)
- moved D2 10.0 mm to (130.8, 81.5), turned to 90 degrees
- moved J1 10.0 mm to (139.8, 75.0)
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Connections:
- D3 pad 1: /GPIO16 -> Net-(D3-Pad1)
- D3 pad 2: Net-(D3-Pad2) -> +3.3VA
- D5 pad 1: GND -> Net-(D5-Pad1)
- D5 pad 2: Net-(D5-Pad2) -> +12V
- R3 pad 1: +3.3VA -> /RST
- R3 pad 2: /RST -> +3.3VA
- R6 pad 1: +3.3VA -> Net-(D3-Pad1)
- R6 pad 2: Net-(D3-Pad2) -> /GPIO16
- R9 pad 1: Net-(D5-Pad2) -> GND
- R9 pad 2: +12V -> Net-(D5-Pad1)
Routing:
- net +12V: track 129.4 -> 56.3 mm
- net GND: track 51.5 -> 113.0 mm, vias 26 -> 20
- net /GPIO5: track 6.59 -> 56.4 mm
- net /GPIO16: track 7.90 -> 27.2 mm, vias 0 -> 2
- net /0VA: track 150.8 -> 133.9 mm
- net Net-(R7-Pad2): track 39.2 -> 55.7 mm
- net /GPIO13: track 35.7 -> 22.9 mm
- net /ADC: track 19.2 -> 11.2 mm
- net /RST: track 14.5 -> 6.84 mm
- net /EN: track 6.61 -> 3.11 mm
- net Net-(D5-Pad2): track 2.81 -> 0.00 mm
- net Net-(D5-Pad1): track 0.00 -> 2.38 mm
- net Net-(R13-Pad2): track 16.3 -> 13.9 mm
- net Net-(D3-Pad1): track 0.00 -> 2.03 mm
- net +5V: track 14.4 -> 12.4 mm
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Other:
- board size 60 x 50 mm -> 50 x 50 mm
- board text added: "JLCJLCJLCJLC"
- board text added: "Revision 0.35"
- board text added: "So, why'd you take this off?"
- board text removed: "104"
- board text removed: "1uF"
- board text removed: "222"
- board text removed: "224"

Commit message: updates... a lot.
Changed lines of the file:
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@@
     (tags resistor)
     (attr smd)
-    (fp_text reference R3 (at -2.25 0 180) (layer F.SilkS)
+    (fp_text reference R3 (at 2.307 0.002 180) (layer F.SilkS)
       (effects (font (size 1 1) (thickness 0.15)))
     )
