File: In Development/LED Timer/LED Timer/LED Timer.sch (KiCad schematic (older format))
At the start: 31 parts, among them J1 Barrel_Jack_Switch, J2 Conn_01x04_Male, J3 Conn_01x03_Female, SW1 DNP, U1 LM7805_TO252-2, U2 ESP-12E

Commit message: added a switch to dectect for soft-reset
Parts:
- added R13: 470, Resistor_SMD:R_0603_1608Metric, symbol Device:R_Small
- added R14: 12K, Resistor_SMD:R_0603_1608Metric, symbol Device:R_Small
- added SW2: SW2, Button_Switch_SMD:SW_SPST_EVQQ2, symbol Switch:SW_Push
Connections:
- net +3.3VA: now also R14.1
- net 0VA: now also SW2.2
- net GPIO12: no longer J2.2 (Pin_2), J2.3 (Pin_3)
- net GPIO13: now also J2.2 (Pin_2), J2.3 (Pin_3)
- net GPIO5: now also R13.1, R14.2
- new net: R13.2, SW2.1
Other:
- moved on the sheet: R7, SW1
Changed lines of the file:
@@
 	1    0    0    -1
 $EndComp
-Text HLabel 6000 1800 0    50   Input ~ 0
-GPIO16
 Wire Wire Line
 	6000 1400 6000 1250
-Wire Wire Line
-	6000 1700 6000 1800
-Text HLabel 6750 1000 1    50   Input ~ 0
-RST
-Wire Wire Line
-	6750 1000 6750 1100
-$Comp
-L Switch:SW_Push SW1
-U 1 1 5ED3BE4B
-P 6750 1500
-F 0 "SW1" V 6704 1648 50  0000 L CNN
-F 1 "DNP" V 6795 1648 50  0000 L CNN
-F 2 "Button_Switch_SMD:SW_SPST_EVQQ2" H 6750 1700 50  0001 C CNN
-F 3 "https://industrial.panasonic.com/ac/cdn/e/control/switch/light-touch/catalog/sw_lt_eng_6s_th.pdf" H 6750 1700 50  0001 C CNN
-F 4 "EVQ-Q2Y03W" V 6750 1500 50  0001 C CNN "Manufacturer Part"
-F 5 "P12961SCT-ND" V 6750 1500 50  0001 C CNN "Digikey Part"
-	1    6750 1500
-	0    1    1    0
-$EndComp
-Wire Wire Line
-	6750 1800 6750 1700
 $Comp
 L Connector:Conn_01x04_Male J2
@@
 	8200 1100 8200 1150
 Text HLabel 8550 1150 2    50   Input ~ 0
-GPIO12
+GPIO13
 Wire Wire Line
 	8200 1150 8550 1150
@@
 $EndComp
 $Comp
-L Device:R_Small R7
-U 1 1 5ED490CD
-P 6750 1200
-F 0 "R7" H 6809 1246 50  0000 L CNN
-F 1 "470" H 6809 1155 50  0000 L CNN
-F 2 "Resistor_SMD:R_0603_1608Metric" H 6750 1200 50  0001 C CNN
-F 3 "https://www.te.com/commerce/DocumentDelivery/DDEController?Action=srchrtrv&DocNm=1773204-3&DocType=DS&DocLang=English" H 6750 1200 50  0001 C CNN
-F 4 "CRGCQ0603J470R" H 6750 1200 50  0001 C CNN "Manufacturer Part"
-F 5 "A130089CT-ND" H 6750 1200 50  0001 C CNN "Digikey Part"
-	1    6750 1200
-	1    0    0    -1
-$EndComp
-$Comp
 L Device:R_Small R8
 U 1 1 5ED49487
@@
 0VA
 Text HLabel 7550 2950 3    50   Input ~ 0
-0VA
-Text HLabel 6750 1800 3    50   Input ~ 0
 0VA
 Text HLabel 2400 3100 1    50   Input ~ 0
@@
 	1    0    0    -1
 $EndComp
+Text HLabel 6650 1800 3    50   Input ~ 0
+0VA
+$Comp
+L Device:R_Small R7
+U 1 1 5ED490CD
+P 6650 1200
+F 0 "R7" H 6709 1246 50  0000 L CNN
+F 1 "470" H 6709 1155 50  0000 L CNN
+F 2 "Resistor_SMD:R_0603_1608Metric" H 6650 1200 50  0001 C CNN
+F 3 "https://www.te.com/commerce/DocumentDelivery/DDEController?Action=srchrtrv&DocNm=1773204-3&DocType=DS&DocLang=English" H 6650 1200 50  0001 C CNN
+F 4 "CRGCQ0603J470R" H 6650 1200 50  0001 C CNN "Manufacturer Part"
+F 5 "A130089CT-ND" H 6650 1200 50  0001 C CNN "Digikey Part"
+	1    6650 1200
+	1    0    0    -1
+$EndComp
+Wire Wire Line
+	6650 1800 6650 1700
+$Comp
+L Switch:SW_Push SW1
+U 1 1 5ED3BE4B
+P 6650 1500
+F 0 "SW1" V 6604 1648 50  0000 L CNN
+F 1 "DNP" V 6695 1648 50  0000 L CNN
+F 2 "Button_Switch_SMD:SW_SPST_EVQQ2" H 6650 1700 50  0001 C CNN
+F 3 "https://industrial.panasonic.com/ac/cdn/e/control/switch/light-touch/catalog/sw_lt_eng_6s_th.pdf" H 6650 1700 50  0001 C CNN
+F 4 "EVQ-Q2Y03W" V 6650 1500 50  0001 C CNN "Manufacturer Part"
+F 5 "P12961SCT-ND" V 6650 1500 50  0001 C CNN "Digikey Part"
+	1    6650 1500
+	0    1    1    0
+$EndComp
+Wire Wire Line
+	6650 1000 6650 1100
+Text HLabel 6650 1000 1    50   Input ~ 0
+RST
+Text HLabel 7200 1800 3    50   Input ~ 0
+0VA
+$Comp
+L Device:R_Small R13
+U 1 1 5ECF1904
+P 7200 1200
+F 0 "R13" H 7259 1246 50  0000 L CNN
+F 1 "470" H 7259 1155 50  0000 L CNN
+F 2 "Resistor_SMD:R_0603_1608Metric" H 7200 1200 50  0001 C CNN
+F 3 "https://www.te.com/commerce/DocumentDelivery/DDEController?Action=srchrtrv&DocNm=1773204-3&DocType=DS&DocLang=English" H 7200 1200 50  0001 C CNN
+F 4 "CRGCQ0603J470R" H 7200 1200 50  0001 C CNN "Manufacturer Part"
+F 5 "A130089CT-ND" H 7200 1200 50  0001 C CNN "Digikey Part"
+	1    7200 1200
+	1    0    0    -1
+$EndComp
+Wire Wire Line
+	7200 1800 7200 1700
+$Comp
+L Switch:SW_Push SW2
+U 1 1 5ECF190D
+P 7200 1500
+F 0 "SW2" V 7154 1648 50  0000 L CNN
+F 1 "SW2" V 7245 1648 50  0000 L CNN
+F 2 "Button_Switch_SMD:SW_SPST_EVQQ2" H 7200 1700 50  0001 C CNN
+F 3 "https://industrial.panasonic.com/ac/cdn/e/control/switch/light-touch/catalog/sw_lt_eng_6s_th.pdf" H 7200 1700 50  0001 C CNN
+F 4 "EVQ-Q2Y03W" V 7200 1500 50  0001 C CNN "Manufacturer Part"
+F 5 "P12961SCT-ND" V 7200 1500 50  0001 C CNN "Digikey Part"
+	1    7200 1500
+	0    1    1    0
+$EndComp
+Wire Wire Line
+	7200 1000 7200 1100
+Wire Wire Line
+	6000 1700 6000 1800
+Text HLabel 6000 1800 0    50   Input ~ 0
+GPIO16
+$Comp
+L Device:R_Small R14
+U 1 1 5ECFC284
+P 7200 2650
+F 0 "R14" H 7050 2600 50  0000 C CNN
+F 1 "12K" H 7050 2700 50  0000 C CNN
+F 2 "Resistor_SMD:R_0603_1608Metric" H 7200 2650 50  0001 C CNN
+F 3 "https://www.te.com/commerce/DocumentDelivery/DDEController?Action=srchrtrv&DocNm=1773204-3&DocType=DS&DocLang=English" H 7200 2650 50  0001 C CNN
+F 4 "CRGCQ0603F12K" V 7200 2650 50  0001 C CNN "Manufacturer Part"
+F 5 "A129701CT-ND" V 7200 2650 50  0001 C CNN "Digikey Part"
+	1    7200 2650
+	-1   0    0    1
+$EndComp
+Connection ~ 7200 2750
+Text HLabel 7200 2550 0    50   Input ~ 0
+GPIO5
+Text HLabel 7200 1000 1    50   Input ~ 0
+GPIO5
 $EndSCHEMATC

Commit message: mod.
Parts:
- removed D6: Red 2, LED_SMD:LED_0805_2012Metric, symbol Device:LED
- R9: value 470 -> 510; footprint Resistor_SMD:R_0603_1608Metric -> Resistor_SMD:R_0805_2012Metric; Digikey Part A130089CT-ND -> A126372CT-ND; Manufacturer Part CRGCQ0603J470R -> CRG0805F510R
Connections:
- net GND: now also D5.1 (K)
Other:
- moved on the sheet: D4, D5, R9
Changed lines of the file:
@@
 L Device:LED D4
 U 1 1 5ED49A6C
-P 8600 2350
-F 0 "D4" H 8593 2095 50  0000 C CNN
-F 1 "Blue 3.2" H 8593 2186 50  0000 C CNN
-F 2 "LED_SMD:LED_0805_2012Metric" H 8600 2350 50  0001 C CNN
-F 3 "https://katalog.we-online.de/led/datasheet/150080BS75000.pdf" H 8600 2350 50  0001 C CNN
-F 4 "150080BS75000" H 8600 2350 50  0001 C CNN "Manufacturer Part"
-F 5 "732-4982-1-ND" H 8600 2350 50  0001 C CNN "Digikey Part"
-	1    8600 2350
+P 8450 2350
+F 0 "D4" H 8443 2095 50  0000 C CNN
+F 1 "Blue 3.2" H 8443 2186 50  0000 C CNN
+F 2 "LED_SMD:LED_0805_2012Metric" H 8450 2350 50  0001 C CNN
+F 3 "https://katalog.we-online.de/led/datasheet/150080BS75000.pdf" H 8450 2350 50  0001 C CNN
+F 4 "150080BS75000" H 8450 2350 50  0001 C CNN "Manufacturer Part"
+F 5 "732-4982-1-ND" H 8450 2350 50  0001 C CNN "Digikey Part"
+	1    8450 2350
 	-1   0    0    1
 $EndComp
@@
 Connection ~ 4500 4700
 Wire Wire Line
-	9000 2350 8750 2350
-Wire Wire Line
-	8450 2350 8150 2350
-Text HLabel 9000 2350 2    50   Input ~ 0
+	8900 2350 8600 2350
+Wire Wire Line
+	8300 2350 8150 2350
+Text HLabel 8900 2350 2    50   Input ~ 0
 0VA
 $Comp
@@
 L Device:R_Small R9
 U 1 1 5ED6C5A9
-P 7900 1850
-F 0 "R9" V 7704 1850 50  0000 C CNN
-F 1 "470" V 7795 1850 50  0000 C CNN
-F 2 "Resistor_SMD:R_0603_1608Metric" H 7900 1850 50  0001 C CNN
-F 3 "https://www.te.com/commerce/DocumentDelivery/DDEController?Action=srchrtrv&DocNm=1773204-3&DocType=DS&DocLang=English" H 7900 1850 50  0001 C CNN
-F 4 "CRGCQ0603J470R" H 7900 1850 50  0001 C CNN "Manufacturer Part"
-F 5 "A130089CT-ND" H 7900 1850 50  0001 C CNN "Digikey Part"
-	1    7900 1850
+P 8050 1850
+F 0 "R9" V 7854 1850 50  0000 C CNN
+F 1 "510" V 7945 1850 50  0000 C CNN
+F 2 "Resistor_SMD:R_0805_2012Metric" H 8050 1850 50  0001 C CNN
+F 3 "https://www.te.com/commerce/DocumentDelivery/DDEController?Action=srchrtrv&DocNm=1773204&DocType=DS&DocLang=English" H 8050 1850 50  0001 C CNN
+F 4 "CRG0805F510R" H 8050 1850 50  0001 C CNN "Manufacturer Part"
+F 5 " A126372CT-ND" H 8050 1850 50  0001 C CNN "Digikey Part"
+	1    8050 1850
 	0    1    1    0
 $EndComp
@@
 L power:GND #PWR0114
 U 1 1 5ED6CF49
-P 9250 1850
-F 0 "#PWR0114" H 9250 1600 50  0001 C CNN
-F 1 "GND" H 9255 1677 50  0000 C CNN
-F 2 "" H 9250 1850 50  0001 C CNN
-F 3 "" H 9250 1850 50  0001 C CNN
-	1    9250 1850
-	1    0    0    -1
-$EndComp
-$Comp
-L Device:LED D6
-U 1 1 5ED73A7E
-P 8850 1850
-F 0 "D6" H 8843 1595 50  0000 C CNN
-F 1 "Red 2" H 8843 1686 50  0000 C CNN
-F 2 "LED_SMD:LED_0805_2012Metric" H 8850 1850 50  0001 C CNN
-F 3 "https://dammedia.osram.info/media/resource/hires/osram-dam-2493505/LS%20R976.pdf" H 8850 1850 50  0001 C CNN
-F 4 "LS R976-NR-1" H 8850 1850 50  0001 C CNN "Manufacturer Part"
-F 5 "475-1278-1-ND" H 8850 1850 50  0001 C CNN "Digikey Part"
-	1    8850 1850
-	-1   0    0    1
-$EndComp
-Wire Wire Line
-	8500 1850 8700 1850
-Wire Wire Line
-	9000 1850 9250 1850
-Wire Wire Line
-	8000 1850 8200 1850
+P 9000 1850
+F 0 "#PWR0114" H 9000 1600 50  0001 C CNN
+F 1 "GND" H 9005 1677 50  0000 C CNN
+F 2 "" H 9000 1850 50  0001 C CNN
+F 3 "" H 9000 1850 50  0001 C CNN
+	1    9000 1850
+	1    0    0    -1
+$EndComp
+Wire Wire Line
+	8150 1850 8350 1850
 $Comp
 L Device:LED D5
 U 1 1 5ED6FA88
-P 8350 1850
-F 0 "D5" H 8343 1595 50  0000 C CNN
-F 1 "Red 2" H 8343 1686 50  0000 C CNN
-F 2 "LED_SMD:LED_0805_2012Metric" H 8350 1850 50  0001 C CNN
-F 3 "https://dammedia.osram.info/media/resource/hires/osram-dam-2493505/LS%20R976.pdf" H 8350 1850 50  0001 C CNN
-F 4 "LS R976-NR-1" H 8350 1850 50  0001 C CNN "Manufacturer Part"
-F 5 "475-1278-1-ND" H 8350 1850 50  0001 C CNN "Digikey Part"
-	1    8350 1850
+P 8500 1850
+F 0 "D5" H 8493 1595 50  0000 C CNN
+F 1 "Red 2" H 8493 1686 50  0000 C CNN
+F 2 "LED_SMD:LED_0805_2012Metric" H 8500 1850 50  0001 C CNN
+F 3 "https://dammedia.osram.info/media/resource/hires/osram-dam-2493505/LS%20R976.pdf" H 8500 1850 50  0001 C CNN
+F 4 "LS R976-NR-1" H 8500 1850 50  0001 C CNN "Manufacturer Part"
+F 5 "475-1278-1-ND" H 8500 1850 50  0001 C CNN "Digikey Part"
+	1    8500 1850
 	-1   0    0    1
 $EndComp
@@
 L power:+12V #PWR0115
 U 1 1 5ED823DC
-P 7700 1850
-F 0 "#PWR0115" H 7700 1700 50  0001 C CNN
-F 1 "+12V" V 7715 1978 50  0000 L CNN
-F 2 "" H 7700 1850 50  0001 C CNN
-F 3 "" H 7700 1850 50  0001 C CNN
-	1    7700 1850
-	0    -1   -1   0
-$EndComp
-Wire Wire Line
-	7700 1850 7800 1850
+P 7850 1850
+F 0 "#PWR0115" H 7850 1700 50  0001 C CNN
+F 1 "+12V" V 7865 1978 50  0000 L CNN
+F 2 "" H 7850 1850 50  0001 C CNN
+F 3 "" H 7850 1850 50  0001 C CNN
+	1    7850 1850
+	0    -1   -1   0
+$EndComp
+Wire Wire Line
+	7850 1850 7950 1850
 Text Notes 8250 1150 0    50   ~ 0
 Data in
@@
 Text HLabel 7200 1000 1    50   Input ~ 0
 GPIO5
+Wire Wire Line
+	8650 1850 9000 1850
 $EndSCHEMATC

Commit message: In production.
Parts:
- added FID1, FID2, FID3: Fiducial, Fiducial:Fiducial_0.5mm_Mask1mm, symbol Mechanical:Fiducial
- added LOGO1: Logo_Open_Hardware_Small, Custom:OSHWLOGO_TOP_0.2_SC-ver, symbol Graphic:Logo_Open_Hardware_Small
- R1, R14, R2, R3, R4, R5: value 12K -> 10K; Digikey Part A129701CT-ND -> A129700CT-ND; Manufacturer Part CRGCQ0603F12K -> CRGCQ0603F10K
- R6: value 470 -> 22; Digikey Part A130089CT-ND -> P22.0HCT-ND; Manufacturer Part CRGCQ0603J470R -> ERJ-3EKF22R0V
Connections:
- net +12V: now also D5.2 (A); no longer R9.2
- net +3.3VA: now also D3.2 (A), R3.2; no longer R3.1, R6.1
- net GND: now also R9.1; no longer D5.1 (K)
- net GPIO16: now also R6.2; no longer D3.1 (K)
- net RST: now also R3.1; no longer R3.2
- new net: D3.1 (K), R6.1
- new net: D5.1 (K), R9.2
Other:
- moved on the sheet: D3, D5, H1, H2, R9

Commit message: updates... a lot.
Parts:
- R6, R8: value 22 -> 10
Changed lines of the file:
@@
 P 8050 2350
 F 0 "R8" V 8246 2350 50  0000 C CNN
-F 1 "22" V 8155 2350 50  0000 C CNN
+F 1 "10" V 8155 2350 50  0000 C CNN
 F 2 "Resistor_SMD:R_0603_1608Metric" H 8050 2350 50  0001 C CNN
 F 3 "https://industrial.panasonic.com/cdbs/www-data/pdf/RDA0000/AOA0000C304.pdf" H 8050 2350 50  0001 C CNN
@@
 P 6000 1600
 F 0 "R6" H 6100 1650 50  0000 C CNN
-F 1 "22" H 6100 1550 50  0000 C CNN
+F 1 "10" H 6100 1550 50  0000 C CNN
 F 2 "Resistor_SMD:R_0603_1608Metric" H 6000 1600 50  0001 C CNN
 F 3 "https://industrial.panasonic.com/cdbs/www-data/pdf/RDA0000/AOA0000C304.pdf" H 6000 1600 50  0001 C CNN
