File: Releases/MFRC522-NodeMCUv2/v1.3/MFRC522 PCB Nodev2.kicad_pcb (KiCad board)
At the start: 2 copper layers, 120 x 50 mm, 46 parts, among them P1 ESP32 NODEMCU DEVKIT1 LEFT HE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, P2 ESP32 NODEMCU DEVKIT1 RIGHT H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, Q2 Q_NPN_BEC, U1 MFRC522, Y1 27.12 MHz

Commit message: updates... a lot.
Parts:
- moved C4 20.2 mm to (137.9, 65.0), turned to 270 degrees
- moved C3 15.6 mm to (133.5, 65.0), turned to 270 degrees
- moved C6 7.88 mm to (142.9, 78.9)
- moved C9 7.88 mm to (142.9, 76.3)
- moved R3 5.59 mm to (135.8, 62.7)
- moved C1 5.46 mm to (142.9, 81.0)
- moved C2 5.46 mm to (142.9, 87.5)
- moved Y1 5.46 mm to (142.9, 84.2)
Connections:
- P1 pad 10: Net-(P1-Pad10) -> GND
- P2 pad 15: +3V3 -> Net-(P2-Pad15)
- P2 pad 2: /RST -> Net-(P2-Pad2)
- P2 pad 3: Net-(P2-Pad3) -> /RST
- P2 pad 6: Net-(P2-Pad6) -> +3.3VA
- P2 pad 7: /GPIO-TH -> GND
- P2 pad 8: Net-(P2-Pad8) -> /GPIO-TH
- R1 pad 2: +3V3 -> +3.3VA
- R2 pad 2: +3V3 -> +3.3VA
Routing:
- net +3V3: track 90.0 -> 62.4 mm, vias 5 -> 4
- net +3.3VA: track 0.00 -> 13.2 mm
- net GND: track 859.8 -> 852.4 mm, vias 21 -> 20
- net Net-(C2-Pad2): track 15.4 -> 17.5 mm
- net /RST: track 19.9 -> 17.9 mm
- net /GPIO-TH: track 6.27 -> 7.49 mm
- net Net-(LED1-Pad2): track 3.29 -> 4.50 mm
- net Net-(C1-Pad2): track 10.7 -> 10.1 mm
Other:
- board text added: "3.3VB|GND|BZR|SDA|STAT"
- board text added: "MISO|SCK|GND|3.3V"
- board text removed: "BZR"
- board text removed: "MISO|SCK 3.3V"
- board text removed: "SDA|STAT"
