File: Releases/MFRC522-NodeMCUv2/v1.3/MFRC522 PCB Nodev2.sch (KiCad schematic (older format))
At the start: 46 parts, among them P1 ESP32 NODEMCU DEVKIT1 LEFT HE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, P2 ESP32 NODEMCU DEVKIT1 RIGHT H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, Q2 Q_NPN_BEC, U1 MFRC522, Y1 27.12 MHz

Commit message: updates... a lot.
Parts:
- R3: value 24 -> 15
Connections:
- net +3V3: no longer P2.15 (Pin_15), R1.2, R2.2
- net GND: now also P1.10 (Pin_10), P2.7 (Pin_7)
- net GPIO-TH: now also P2.8 (Pin_8); no longer P2.7 (Pin_7)
- net RST: now also P2.3 (Pin_3); no longer P2.2 (Pin_2)
- net +3.3VA: now reaches P2.6 (Pin_6)
- net +3.3VA: now also R1.2, R2.2
- no-connect marks 27 -> 25
Changed lines of the file:
@@
 Text HLabel 1650 1900 2    50   Output ~ 0
 IRQ
-Text HLabel 1650 3500 2    50   Output ~ 0
+Text HLabel 1650 3400 2    50   Output ~ 0
 GPIO-TH
 NoConn ~ 1650 3700
 NoConn ~ 1650 3800
-NoConn ~ 1650 3400
-Text HLabel 1650 4000 2    50   Output ~ 0
+NoConn ~ 1650 4000
+Text HLabel 1650 3900 2    50   Output ~ 0
 RST
 $Comp
@@
 L power:+3.3V #PWR0104
 U 1 1 5EADB5D4
-P 1650 2700
-F 0 "#PWR0104" H 1650 2550 50  0001 C CNN
-F 1 "+3.3V" V 1650 2800 50  0000 L CNN
-F 2 "" H 1650 2700 50  0001 C CNN
-F 3 "" H 1650 2700 50  0001 C CNN
-	1    1650 2700
+P 1650 1300
+F 0 "#PWR0104" H 1650 1150 50  0001 C CNN
+F 1 "+3.3V" V 1650 1400 50  0000 L CNN
+F 2 "" H 1650 1300 50  0001 C CNN
+F 3 "" H 1650 1300 50  0001 C CNN
+	1    1650 1300
+	0    1    1    0
+$EndComp
+$Comp
+L power:GND #PWR0105
+U 1 1 5EADB925
+P 1650 1400
+F 0 "#PWR0105" H 1650 1150 50  0001 C CNN
+F 1 "GND" V 1655 1272 50  0000 R CNN
+F 2 "" H 1650 1400 50  0001 C CNN
+F 3 "" H 1650 1400 50  0001 C CNN
+	1    1650 1400
+	0    -1   -1   0
+$EndComp
+$Comp
+L power:+3.3VA #PWR0106
+U 1 1 5EADC163
+P 1650 3600
+F 0 "#PWR0106" H 1650 3450 50  0001 C CNN
+F 1 "+3.3VA" V 1665 3728 50  0000 L CNN
+F 2 "" H 1650 3600 50  0001 C CNN
+F 3 "" H 1650 3600 50  0001 C CNN
+	1    1650 3600
 	0    1    1    0
 $EndComp
@@
 	1    0    0    -1
 $EndComp
+$Comp
+L power:+3.3VA #PWR0117
+U 1 1 5EB0AB02
+P 3700 3800
+F 0 "#PWR0117" H 3700 3650 50  0001 C CNN
+F 1 "+3.3VA" H 3715 3973 50  0000 C CNN
+F 2 "" H 3700 3800 50  0001 C CNN
+F 3 "" H 3700 3800 50  0001 C CNN
+	1    3700 3800
+	-1   0    0    1
+$EndComp
 Wire Wire Line
 	3700 3700 3700 3800
@@
 $EndComp
 $Comp
+L power:GND #PWR0125
+U 1 1 5EADBE51
+P 1650 3500
+F 0 "#PWR0125" H 1650 3250 50  0001 C CNN
+F 1 "GND" V 1655 3372 50  0000 R CNN
+F 2 "" H 1650 3500 50  0001 C CNN
+F 3 "" H 1650 3500 50  0001 C CNN
+	1    1650 3500
+	0    -1   -1   0
+$EndComp
+$Comp
 L power:GND #PWR0126
 U 1 1 5EADBBCC
@@
 NoConn ~ 1650 3100
 NoConn ~ 1650 3000
+NoConn ~ 1650 2700
 NoConn ~ 1650 2900
 Wire Wire Line
@@
 	-1   0    0    1
 $EndComp
+$Comp
+L power:+3.3VA #PWR0109
+U 1 1 5F0B1F2D
+P 5650 2450
+F 0 "#PWR0109" H 5650 2300 50  0001 C CNN
+F 1 "+3.3VA" V 5665 2577 50  0000 L CNN
+F 2 "" H 5650 2450 50  0001 C CNN
+F 3 "" H 5650 2450 50  0001 C CNN
+	1    5650 2450
+	0    -1   -1   0
+$EndComp
 Text Notes 7350 7500 0    75   ~ 0
 MFRC522 board for Innexgo LLC
@@
 P 1500 5900
 F 0 "R3" H 1559 5946 50  0000 L CNN
-F 1 "24" H 1559 5855 50  0000 L CNN
+F 1 "15" H 1559 5855 50  0000 L CNN
 F 2 "Resistor_SMD:R_0603_1608Metric" H 1500 5900 50  0001 C CNN
 F 3 "~" H 1500 5900 50  0001 C CNN
@@
 Wire Wire Line
 	8450 4150 8550 4150
-NoConn ~ 1650 3600
-NoConn ~ 1650 3900
-$Comp
-L power:+3.3V #PWR0106
-U 1 1 5F0CE5E6
-P 1650 1300
-F 0 "#PWR0106" H 1650 1150 50  0001 C CNN
-F 1 "+3.3V" V 1650 1400 50  0000 L CNN
-F 2 "" H 1650 1300 50  0001 C CNN
-F 3 "" H 1650 1300 50  0001 C CNN
-	1    1650 1300
-	0    1    1    0
-$EndComp
-NoConn ~ 1650 1400
-$Comp
-L power:+3.3V #PWR?
-U 1 1 5F09AE72
-P 5650 2450
-F 0 "#PWR?" H 5650 2300 50  0001 C CNN
-F 1 "+3.3V" V 5665 2578 50  0000 L CNN
-F 2 "" H 5650 2450 50  0001 C CNN
-F 3 "" H 5650 2450 50  0001 C CNN
-	1    5650 2450
-	0    -1   -1   0
-$EndComp
-$Comp
-L power:+3.3V #PWR?
-U 1 1 5F09B301
-P 3700 3800
-F 0 "#PWR?" H 3700 3650 50  0001 C CNN
-F 1 "+3.3V" H 3715 3928 50  0000 L CNN
-F 2 "" H 3700 3800 50  0001 C CNN
-F 3 "" H 3700 3800 50  0001 C CNN
-	1    3700 3800
-	-1   0    0    1
-$EndComp
 $EndSCHEMATC
