File: Releases/MFRC522-ESP32/MFRC522 PCB ESP32.sch (KiCad schematic (older format))
At the start: 51 parts, among them P1 ESP32 DEVKIT1 LEFT HEADER-MAL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, P2 ESP32 DEVKIT1 RIGHT HEADER-MA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, Q2 Q_NPN_BEC, U1 MFRC522, Y1 27.12 MHz

Commit message: mfrc522 v2 80x80 laid out
Parts:
- added R20: R_Axial, Resistor_THT:R_Axial_DIN0309_L9.0mm_D3.2mm_P12.70mm_Horizontal, symbol Device:R_Small
Connections:
- net +3V3: now also R20.2
- net GPIO-TH: now also P2.7 (Pin_7); no longer P2.9 (Pin_9)
- net IRQ: now also P1.9 (Pin_9); no longer P1.13 (Pin_13)
- net RST: now also P2.2 (Pin_2); no longer P2.10 (Pin_10)
- net SDA: now also P2.9 (Pin_9); no longer P1.9 (Pin_9)
- net STATUS1: now also P1.13 (Pin_13); no longer P2.2 (Pin_2)
- net STATUS2: now also P2.10 (Pin_10); no longer P2.7 (Pin_7)
- net at BZ1.1 (-), D1.1 (K), R14.2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: now also R20.1
Changed lines of the file:
@@
 NoConn ~ 1650 2200
 NoConn ~ 1650 2300
-Text HLabel 1650 1100 2    50   Output ~ 0
+Text HLabel 1650 1500 2    50   Output ~ 0
 IRQ
-Text HLabel 1650 3300 2    50   Output ~ 0
+Text HLabel 1650 3500 2    50   Output ~ 0
 GPIO-TH
 NoConn ~ 1650 3700
 NoConn ~ 1650 3800
 NoConn ~ 1650 3400
-Text HLabel 1650 3200 2    50   Output ~ 0
+Text HLabel 1650 4000 2    50   Output ~ 0
 RST
 $Comp
@@
 	0    -1   -1   0
 $EndComp
-Text HLabel 1650 1500 2    50   BiDi ~ 0
+Text HLabel 1650 3300 2    50   BiDi ~ 0
 SDA
 NoConn ~ 1650 2000
@@
 	1    0    0    -1
 $EndComp
+$Comp
+L Device:R_Small R20
+U 1 1 5EDE0E89
+P 8350 3850
+F 0 "R20" V 8154 3850 50  0000 C CNN
+F 1 "R_Axial" V 8245 3850 50  0000 C CNN
+F 2 "Resistor_THT:R_Axial_DIN0309_L9.0mm_D3.2mm_P12.70mm_Horizontal" H 8350 3850 50  0001 C CNN
+F 3 "~" H 8350 3850 50  0001 C CNN
+	1    8350 3850
+	0    1    1    0
+$EndComp
 Connection ~ 8150 4450
 Wire Wire Line
 	8150 4450 8250 4450
+Wire Wire Line
+	8550 3850 8550 4150
 Connection ~ 8550 4450
 Wire Wire Line
 	8550 4450 8800 4450
+Wire Wire Line
+	8450 3850 8550 3850
 NoConn ~ 1650 3600
 NoConn ~ 1650 3900
@@
 Wire Wire Line
 	3000 6750 3000 6900
-Text HLabel 1650 4000 2    50   Input ~ 0
+Text HLabel 1650 1100 2    50   Input ~ 0
 STATUS1
 $Comp
@@
 	1    0    0    -1
 $EndComp
-Text HLabel 1650 3500 2    50   Output ~ 0
+Text HLabel 1650 3200 2    50   Output ~ 0
 STATUS2
 Text HLabel 2300 5950 1    50   Input ~ 0
@@
 Wire Wire Line
 	3000 6350 3000 6450
+Wire Wire Line
+	8150 3850 8150 4150
+Wire Wire Line
+	8250 3850 8150 3850
 $Comp
 L Device:R_Small R21
@@
 Wire Wire Line
 	8450 4150 8550 4150
+Connection ~ 8550 4150
 Wire Wire Line
 	8550 4150 8550 4450
 Wire Wire Line
 	8250 4150 8150 4150
+Connection ~ 8150 4150
 Wire Wire Line
 	8150 4150 8150 4450
